File: ergogen/pcbs/ergojodi.kicad_pcb (KiCad board)
At the start: 2 copper layers, 261.4 x 115 mm, 76 parts

Commit message: Routed the PCB
Parts:
- removed XX1, XX4: , MODULE_102010428
- added REF**: MODULE_102010428, MODULE_102010428, F.Cu at (223.8, 100.2)
- added REF**: MODULE_102010428, MODULE_102010428, F.Cu at (197.5, 100.2)
- added REF**: BreakLine_5h_D0.5mm_P0.85mm, Panelization:BreakLine_5h_D0.5mm_P0.85mm, F.Cu at (213.3, 102.0)
- added REF**: BreakLine_5h_D0.5mm_P0.85mm, Panelization:BreakLine_5h_D0.5mm_P0.85mm, F.Cu at (208.0, 102.0)
- moved D35 13.0 mm to (245.2, 177.1)
- moved S35 13.0 mm to (242.7, 172.7)
- moved S19 13.0 mm to (319.9, 150.0)
- moved S20 13.0 mm to (321.2, 131.0)
- moved S21 13.0 mm to (322.6, 112.1)
- moved D19 13.0 mm to (319.6, 155.0)
- moved D20 13.0 mm to (320.9, 136.0)
- moved D21 13.0 mm to (322.2, 117.1)
- moved D34 13.0 mm to (263.6, 169.3)
- moved D31 13.0 mm to (243.3, 146.5)
- moved D32 13.0 mm to (243.3, 127.5)
- moved D33 13.0 mm to (243.3, 108.5)
- moved S31 13.0 mm to (243.3, 141.5)
- moved S32 13.0 mm to (243.3, 122.5)
- moved S33 13.0 mm to (243.3, 103.5)
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Routing:
- net l_A10: track 0.00 -> 176.7 mm, vias 0 -> 1
- net l_A8: track 0.00 -> 161.5 mm, vias 0 -> 1
- net r_A0: track 0.00 -> 158.6 mm, vias 0 -> 1
- net l_A2: track 0.00 -> 158.6 mm
- net r_A8: track 0.00 -> 147.7 mm
- net l_A7: track 0.00 -> 144.6 mm, vias 0 -> 1
- net l_A9: track 0.00 -> 143.7 mm, vias 0 -> 1
- net r_A2: track 0.00 -> 143.3 mm, vias 0 -> 1
- net l_A1: track 0.00 -> 142.2 mm
- net l_A0: track 0.00 -> 136.4 mm
- net r_A9: track 0.00 -> 134.6 mm
- net l_A3: track 0.00 -> 134.0 mm
- net r_A1: track 0.00 -> 125.5 mm, vias 0 -> 1
- net r_A3: track 0.00 -> 125.4 mm, vias 0 -> 1
- net l_A4: track 0.00 -> 125.0 mm, vias 0 -> 1
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Other:
- board size 261.4 x 115 mm -> 247 x 115 mm
- net class Default removed
